Commit message: Create s1_description  s1_body.urdf.xacro

File: s1_description/urdf/s1_body.urdf.xacro (robot description, xacro)
@@ -29,5 +29,5 @@
   <link name="left_wheel_link" >
     <visual>
-      <origin xyz="${wheel_left_pos}" rpy="0 1.5707 1.5707" />
+      <origin xyz="0 0 0" rpy="0 1.5707 1.5707" />
         <geometry>
           <mesh filename="package://s1_description/meshes/wheel.dae"/>
@@ -38,5 +38,5 @@
       </visual>
     <inertial>
-      <origin xyz="${wheel_left_pos}"/>
+      <origin xyz="0 0 0"/>
       <mass value="0.01" />
       <inertia ixx="0.001" ixy="0.0" ixz="0.0"
@@ -44,5 +44,5 @@
     </inertial>
     <collision>
-      <origin xyz="${wheel_left_pos}" rpy="0 1.5707 1.5707" />
+      <origin xyz="0 0 0" rpy="0 1.5707 1.5707" />
       <geometry>
         <cylinder radius="${wheel_radius}" length = "${wheel_length}"/>
@@ -58,5 +58,5 @@
   <link name="right_wheel_link" >
     <visual>
-      <origin xyz="${wheel_right_pos}" rpy="0 1.5707 1.5707" />
+      <origin xyz="0 0 0" rpy="0 1.5707 1.5707" />
         <geometry>
           <mesh filename="package://s1_description/meshes/wheel.dae"/>
@@ -67,5 +67,5 @@
       </visual>
     <inertial>
-      <origin xyz="${wheel_right_pos}"/>
+      <origin xyz="0 0 0 "/>
       <mass value="0.01" />
       <inertia ixx="0.001" ixy="0.0" ixz="0.0"
@@ -73,5 +73,5 @@
     </inertial>
     <collision>
-      <origin xyz="${wheel_right_pos}" rpy="0 1.5707 1.5707" />
+      <origin xyz="0 0 0" rpy="0 1.5707 1.5707" />
       <geometry>
         <cylinder radius="${wheel_radius}" length = "${wheel_length}"/>
